Commit message: feat: update so101_control package with hardware interface and ROS2 control configuration

File: ros2_ws/so101_control/config/so101.ros2_control.xacro (robot description, xacro)
@@ -1,14 +1,6 @@
 <?xml version="1.0"?>
 <robot xmlns:xacro="http://www.ros.org/wiki/xacro">
-    <xacro:macro name="so101_ros2_control" params="name use_mock_hardware">
+    <xacro:macro name="so101_ros2_control" params="name use_mock_hardware use_gazebo">
     <ros2_control name="${name}" type="system">
-      <xacro:unless value="${use_mock_hardware}">
-        <hardware>
-            <plugin>so101_control/so101_hardware_interface</plugin>
-            <param name="usb_port">/dev/ttyACM0</param>
-            <param name="baud_rate">1000000</param>
-            <param name="control_mode">0</param>
-        </hardware>
-      </xacro:unless>
       <xacro:if value="${use_mock_hardware}">
         <hardware>
@@ -16,4 +8,17 @@
         </hardware>
       </xacro:if>
+      <xacro:unless value="${use_mock_hardware}">
+        <hardware>
+          <xacro:if value="${use_gazebo}">
+            <plugin>gz_ros2_control/GazeboSimSystem</plugin>
+          </xacro:if>
+          <xacro:unless value="${use_gazebo}">
+            <plugin>so101_control/so101_hardware_interface</plugin>
+            <param name="usb_port">/dev/ttyACM0</param>
+            <param name="baud_rate">1000000</param>
+            <param name="control_mode">0</param>
+          </xacro:unless>
+        </hardware>
+      </xacro:unless>
         <joint name="shoulder_pan">
             <param name="id">1</param>

File: ros2_ws/so101_control/config/so101.urdf.xacro (robot description, xacro)
@@ -1,9 +1,26 @@
 <?xml version="1.0"?>
 <robot xmlns:xacro="http://www.ros.org/wiki/xacro" name="so101_robot">
-  <xacro:arg name="use_mock_hardware" default="false" />
+  <xacro:arg name="use_mock_hardware" default="true" />
+  <xacro:arg name="use_gazebo" default="true" />
+  <xacro:arg name="controller_config_file" default="$(find so101_control)/config/so101.yaml" />
+  <!-- Fixed world link for clamping -->
+  <link name="world"/>
   <xacro:include filename="$(find so101_description)/urdf/so101_description.urdf.xacro" />
   <xacro:so101_new_calib/>
+  <!-- Clamp base_link to world (Gazebo will handle this as floating base constraint) -->
+  <joint name="world_base_joint" type="fixed">
+    <parent link="world"/>
+    <child link="base_link"/>
+    <origin xyz="0 0 0" rpy="0 0 0"/>
+  </joint>
   <xacro:include filename="$(find so101_control)/config/so101.ros2_control.xacro" />
   <xacro:so101_ros2_control
-    name="so101" use_mock_hardware="$(arg use_mock_hardware)"/>
+    name="so101" use_mock_hardware="$(arg use_mock_hardware)" use_gazebo="$(arg use_gazebo)"/>
+  <xacro:if value="$(arg use_gazebo)">
+    <gazebo>
+      <plugin filename="libgz_ros2_control-system.so" name="gz_ros2_control::GazeboSimROS2ControlPlugin">
+        <parameters>$(arg controller_config_file)</parameters>
+      </plugin>
+    </gazebo>
+  </xacro:if>
 </robot>
